File: protoboard-double/protoboard-double.kicad_pcb (KiCad board)
At the start: 2 copper layers, 50.8 x 58.4 mm, 23 parts, among them J1 MODULE_HEADER, J2 MODULE_HEADER, P1 CONN_01X22, P10 CONN_01X22, P11 CONN_01X22, P12 CONN_01X22, P13 CONN_01X22, P14 CONN_01X22, P15 CONN_01X22, P16 CONN_01X22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

Commit message: gerbers and zip
Other:
- rule pad_to_mask_clearance: 0 -> 0.0762
Changed lines of the file:
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@@
     (pad_size 1.5 1.5)
     (pad_drill 0.6)
-    (pad_to_mask_clearance 0)
+    (pad_to_mask_clearance 0.0762)
     (aux_axis_origin 101.6 127)
     (grid_origin 101.6 127)
     (visible_elements FFFFFF7F)
     (pcbplotparams
-      (layerselection 0x00030_80000001)
+      (layerselection 0x010f0_80000001)
       (usegerberextensions false)
       (excludeedgelayer true)
@@
       (plotinvisibletext false)
       (padsonsilk false)
-      (subtractmaskfromsilk false)
+      (subtractmaskfromsilk true)
       (outputformat 1)
       (mirror false)
-      (drillshape 1)
+      (drillshape 0)
       (scaleselection 1)
-      (outputdirectory ""))
+      (outputdirectory gerbers/))
   )
   (net 0 "")

Commit message: doublewide ready for production
Parts:
- SILK1: footprint parts:TESSEL-HEXAGON-LOGO -> parts:TESSEL-HEXAGON-LOGO-BACK; moved to B.Cu
- moved SILK1 10.2 mm to (118.7, 97.8), turned to 270 degrees
- moved P11 0.64 mm to (129.5, 97.8)
- moved P15 0.64 mm to (139.7, 97.8)
- moved P18 0.64 mm to (147.3, 97.8)
- moved P10 0.64 mm to (127.0, 97.8)
- moved P2 0.64 mm to (114.3, 97.8)
- moved P3 0.64 mm to (109.2, 97.8)
- moved P5 0.64 mm to (119.4, 97.8)
- moved P7 0.64 mm to (121.9, 97.8)
- moved P8 0.64 mm to (124.5, 97.8)
- moved P1 0.63 mm to (111.8, 97.8)
- moved P12 0.63 mm to (132.1, 97.8)
- moved P13 0.63 mm to (134.6, 97.8)
- moved P14 0.63 mm to (137.2, 97.8)
- moved P16 0.63 mm to (142.2, 97.8)
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Routing:
- net Net-(C1-Pad2): track 159.7 -> 157.2 mm
- net Net-(J1-Pad1): track 89.1 -> 88.5 mm
- net Net-(J2-Pad9): track 6.35 -> 5.72 mm
- net Net-(J2-Pad8): track 6.35 -> 5.72 mm
- net Net-(J2-Pad7): track 6.35 -> 5.72 mm
- net Net-(J2-Pad6): track 6.35 -> 5.72 mm
- net Net-(J2-Pad5): track 6.35 -> 5.72 mm
- net Net-(J2-Pad4): track 6.35 -> 5.72 mm
- net Net-(J2-Pad3): track 6.35 -> 5.72 mm
- net Net-(J2-Pad10): track 6.35 -> 5.72 mm
- net Net-(J1-Pad9): track 6.35 -> 5.72 mm
- net Net-(J1-Pad8): track 6.35 -> 5.72 mm
- net Net-(J1-Pad7): track 6.35 -> 5.72 mm
- net Net-(J1-Pad6): track 6.35 -> 5.72 mm
- net Net-(J1-Pad5): track 6.35 -> 5.72 mm
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Other:
- board text added: "TM-15-01"
- board text added: "diy-module"
- board text added: "tessel.io"

Commit message: feedback incorporated for doublewide. all aboard the PCB ship!
Parts:
- added P20: CONN_01X10, parts:1x10_BIG, F.Cu at (106.7, 82.5)
- added P21: CONN_01X10, parts:1x10_BIG, F.Cu at (108.0, 113.0)
- added P22: CONN_01X10, parts:1x10_BIG, F.Cu at (108.0, 82.5)
- J1, J2: footprint parts:MODULE_HEADER_MODULE -> parts:MODULE_HEADER_MODULE_BIG
- P1, P10, P11, P12, P13, P14, P15, P16, P17, P18, P19, P2, P4, P5, P7, P8: footprint parts:1x22 -> parts:1x22_BIG
- P3, P6, P9: value CONN_01X22 -> CONN_01X10; footprint parts:1x22 -> parts:1x10_BIG
- SILK1: footprint parts:TESSEL-HEXAGON-LOGO-BACK -> parts:TESSEL-HEXAGON-LOGO-BACK-BIG
- moved P6 15.3 mm to (109.2, 82.5)
- moved P3 15.2 mm to (109.2, 113.0)
- moved P9 15.2 mm to (106.7, 113.0)
- moved SILK1 8.25 mm to (127.0, 97.8)
Connections:
- P1 pad 11: Net-(P1-Pad11) -> Net-(C1-Pad1)
- P1 pad 12: Net-(P1-Pad12) -> Net-(C1-Pad2)
- P10 pad 11: Net-(P10-Pad11) -> Net-(C1-Pad1)
- P10 pad 12: Net-(P10-Pad12) -> Net-(C1-Pad2)
- P11 pad 11: Net-(P11-Pad11) -> Net-(C1-Pad1)
- P11 pad 12: Net-(P11-Pad12) -> Net-(C1-Pad2)
- P12 pad 11: Net-(P12-Pad11) -> Net-(C1-Pad1)
- P12 pad 12: Net-(P12-Pad12) -> Net-(C1-Pad2)
- P13 pad 11: Net-(P13-Pad11) -> Net-(C1-Pad1)
- P13 pad 12: Net-(P13-Pad12) -> Net-(C1-Pad2)
- P14 pad 11: Net-(P14-Pad11) -> Net-(C1-Pad1)
- P14 pad 12: Net-(P14-Pad12) -> Net-(C1-Pad2)
- P15 pad 11: Net-(P15-Pad11) -> Net-(C1-Pad1)
- P15 pad 12: Net-(P15-Pad12) -> Net-(C1-Pad2)
- P16 pad 11: Net-(P16-Pad11) -> Net-(C1-Pad1)
- P16 pad 12: Net-(P16-Pad12) -> Net-(C1-Pad2)
- P17 pad 11: Net-(P17-Pad11) -> Net-(C1-Pad1)
- P17 pad 12: Net-(P17-Pad12) -> Net-(C1-Pad2)
- P18 pad 11: Net-(P18-Pad11) -> Net-(C1-Pad1)
- P18 pad 12: Net-(P18-Pad12) -> Net-(C1-Pad2)
- P19 pad 11: Net-(P19-Pad11) -> Net-(C1-Pad1)
- P19 pad 12: Net-(P19-Pad12) -> Net-(C1-Pad2)
- P2 pad 11: Net-(P2-Pad11) -> Net-(C1-Pad1)
- P2 pad 12: Net-(P2-Pad12) -> Net-(C1-Pad2)
- P4 pad 11: Net-(P4-Pad11) -> Net-(C1-Pad1)
- P4 pad 12: Net-(P4-Pad12) -> Net-(C1-Pad2)
- P5 pad 11: Net-(P5-Pad11) -> Net-(C1-Pad1)
- P5 pad 12: Net-(P5-Pad12) -> Net-(C1-Pad2)
- P6 pad 1: Net-(J1-Pad1) -> Net-(C1-Pad1)
- P6 pad 10: Net-(J1-Pad10) -> Net-(J2-Pad10)
- P6 pad 2: Net-(J1-Pad2) -> Net-(C1-Pad2)
- P6 pad 3: Net-(J1-Pad3) -> Net-(J2-Pad3)
- P6 pad 4: Net-(J1-Pad4) -> Net-(J2-Pad4)
- P6 pad 5: Net-(J1-Pad5) -> Net-(J2-Pad5)
- P6 pad 6: Net-(J1-Pad6) -> Net-(J2-Pad6)
- P6 pad 7: Net-(J1-Pad7) -> Net-(J2-Pad7)
- P6 pad 8: Net-(J1-Pad8) -> Net-(J2-Pad8)
- P6 pad 9: Net-(J1-Pad9) -> Net-(J2-Pad9)
- P7 pad 11: Net-(P7-Pad11) -> Net-(C1-Pad1)
- P7 pad 12: Net-(P7-Pad12) -> Net-(C1-Pad2)
- P8 pad 11: Net-(P8-Pad11) -> Net-(C1-Pad1)
- P8 pad 12: Net-(P8-Pad12) -> Net-(C1-Pad2)
Routing:
- net Net-(J1-Pad2): track 145.1 -> 5.72 mm
- net Net-(C1-Pad2): track 157.2 -> 246.0 mm
- net Net-(P3-Pad12): track 3.81 -> 0.00 mm
- net Net-(C1-Pad1): track 99.1 -> 102.7 mm
- net Net-(P3-Pad11): track 2.54 -> 0.00 mm
Other:
- board text added: "diy- module"
- board text removed: "diy-module"
