File: protoboard-single/protoboard-single.sch (KiCad schematic (older format))
At the start: 16 parts, among them J1 MODULE_HEADER, J10 MODULE_HEADER, J11 MODULE_HEADER, J12 MODULE_HEADER, J13 MODULE_HEADER, J14 MODULE_HEADER, J15 MODULE_HEADER, J2 MODULE_HEADER, J3 MODULE_HEADER, J4 MODULE_HEADER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

Commit message: production-ready files?
Parts:
- SILK1: footprint parts:TESSEL-HEXAGON-LOGO -> parts:TESSEL-HEXAGON-LOGO-BACK
Changed lines of the file:
@@
 F 0 "SILK1" H 3900 2850 60  0000 C CNN
 F 1 "logo" H 3900 2750 60  0000 C CNN
-F 2 "parts:TESSEL-HEXAGON-LOGO" H 3900 2800 60  0001 C CNN
+F 2 "parts:TESSEL-HEXAGON-LOGO-BACK" H 3900 2800 60  0001 C CNN
 F 3 "" H 3900 2800 60  0000 C CNN
 	1    3900 2800

Commit message: feedback incorporated for doublewide. all aboard the PCB ship!
Parts:
- J1: footprint parts:MODULE_HEADER_MODULE -> parts:MODULE_HEADER_MODULE_BIG
- J10, J11, J12, J13, J14, J15, J2, J3, J4, J5, J6, J7, J8, J9: footprint parts:1x10 -> parts:1x10_BIG
Changed lines of the file:
@@
 F 0 "J1" H 5050 3350 60  0000 C CNN
 F 1 "MODULE_HEADER" V 5100 2750 60  0000 C CNN
-F 2 "parts:MODULE_HEADER_MODULE" H 5400 2800 60  0001 C CNN
+F 2 "parts:MODULE_HEADER_MODULE_BIG" H 5400 2800 60  0001 C CNN
 F 3 "" H 5400 2800 60  0000 C CNN
 	1    5400 2800
@@
 F 0 "J5" H 3100 6300 60  0000 C CNN
 F 1 "MODULE_HEADER" V 3150 5700 60  0000 C CNN
-F 2 "parts:1x10" H 3450 5750 60  0001 C CNN
+F 2 "parts:1x10_BIG" H 3450 5750 60  0001 C CNN
 F 3 "" H 3450 5750 60  0000 C CNN
 	1    3450 5750
@@
 F 0 "J6" H 3950 6300 60  0000 C CNN
 F 1 "MODULE_HEADER" V 4000 5700 60  0000 C CNN
-F 2 "parts:1x10" H 4300 5750 60  0001 C CNN
+F 2 "parts:1x10_BIG" H 4300 5750 60  0001 C CNN
 F 3 "" H 4300 5750 60  0000 C CNN
 	1    4300 5750
@@
 F 0 "J7" H 4800 6300 60  0000 C CNN
 F 1 "MODULE_HEADER" V 4850 5700 60  0000 C CNN
-F 2 "parts:1x10" H 5150 5750 60  0001 C CNN
+F 2 "parts:1x10_BIG" H 5150 5750 60  0001 C CNN
 F 3 "" H 5150 5750 60  0000 C CNN
 	1    5150 5750
@@
 F 0 "J8" H 5650 6300 60  0000 C CNN
 F 1 "MODULE_HEADER" V 5700 5700 60  0000 C CNN
-F 2 "parts:1x10" H 6000 5750 60  0001 C CNN
+F 2 "parts:1x10_BIG" H 6000 5750 60  0001 C CNN
 F 3 "" H 6000 5750 60  0000 C CNN
 	1    6000 5750
@@
 F 0 "J9" H 6500 6300 60  0000 C CNN
 F 1 "MODULE_HEADER" V 6550 5700 60  0000 C CNN
-F 2 "parts:1x10" H 6850 5750 60  0001 C CNN
+F 2 "parts:1x10_BIG" H 6850 5750 60  0001 C CNN
 F 3 "" H 6850 5750 60  0000 C CNN
 	1    6850 5750
@@
 F 0 "J10" H 7350 6300 60  0000 C CNN
 F 1 "MODULE_HEADER" V 7400 5700 60  0000 C CNN
-F 2 "parts:1x10" H 7700 5750 60  0001 C CNN
+F 2 "parts:1x10_BIG" H 7700 5750 60  0001 C CNN
 F 3 "" H 7700 5750 60  0000 C CNN
 	1    7700 5750
@@
 F 0 "J11" H 8200 6300 60  0000 C CNN
 F 1 "MODULE_HEADER" V 8250 5700 60  0000 C CNN
-F 2 "parts:1x10" H 8550 5750 60  0001 C CNN
+F 2 "parts:1x10_BIG" H 8550 5750 60  0001 C CNN
 F 3 "" H 8550 5750 60  0000 C CNN
 	1    8550 5750
@@
 F 0 "J12" H 9050 6300 60  0000 C CNN
 F 1 "MODULE_HEADER" V 9100 5700 60  0000 C CNN
-F 2 "parts:1x10" H 9400 5750 60  0001 C CNN
+F 2 "parts:1x10_BIG" H 9400 5750 60  0001 C CNN
 F 3 "" H 9400 5750 60  0000 C CNN
 	1    9400 5750
@@
 F 0 "J2" H 6700 3350 60  0000 C CNN
 F 1 "MODULE_HEADER" V 6750 2750 60  0000 C CNN
-F 2 "parts:1x10" H 7050 2800 60  0001 C CNN
+F 2 "parts:1x10_BIG" H 7050 2800 60  0001 C CNN
 F 3 "" H 7050 2800 60  0000 C CNN
 	1    7050 2800
@@
 F 0 "J3" H 1400 6300 60  0000 C CNN
 F 1 "MODULE_HEADER" V 1450 5700 60  0000 C CNN
-F 2 "parts:1x10" H 1750 5750 60  0001 C CNN
+F 2 "parts:1x10_BIG" H 1750 5750 60  0001 C CNN
 F 3 "" H 1750 5750 60  0000 C CNN
 	1    1750 5750
@@
 F 0 "J4" H 2250 6300 60  0000 C CNN
 F 1 "MODULE_HEADER" V 2300 5700 60  0000 C CNN
-F 2 "parts:1x10" H 2600 5750 60  0001 C CNN
+F 2 "parts:1x10_BIG" H 2600 5750 60  0001 C CNN
 F 3 "" H 2600 5750 60  0000 C CNN
 	1    2600 5750
@@
 F 0 "J13" H 9850 6300 60  0000 C CNN
 F 1 "MODULE_HEADER" V 9900 5700 60  0000 C CNN
-F 2 "parts:1x10" H 10200 5750 60  0001 C CNN
+F 2 "parts:1x10_BIG" H 10200 5750 60  0001 C CNN
 F 3 "" H 10200 5750 60  0000 C CNN
 	1    10200 5750
@@
 F 0 "J14" H 5850 3350 60  0000 C CNN
 F 1 "MODULE_HEADER" V 5900 2750 60  0000 C CNN
-F 2 "parts:1x10" H 6200 2800 60  0001 C CNN
+F 2 "parts:1x10_BIG" H 6200 2800 60  0001 C CNN
 F 3 "" H 6200 2800 60  0000 C CNN
 	1    6200 2800
@@
 F 0 "J15" H 7500 3350 60  0000 C CNN
 F 1 "MODULE_HEADER" V 7550 2750 60  0000 C CNN
-F 2 "parts:1x10" H 7850 2800 60  0001 C CNN
+F 2 "parts:1x10_BIG" H 7850 2800 60  0001 C CNN
 F 3 "" H 7850 2800 60  0000 C CNN
 	1    7850 2800
